Commit message: Przebuduj pliki startowe; dodaj węzeł kontrolera obrotu i pochylenia; zaktualizuj świat lidar_test o symulacyjne kule

File: src/ugv_description/urdf/ugv_beast.urdf (robot description, URDF)
Before this commit: robot ugv_beast, 19 links, 18 joints
Joints:
- joint pt_base_link_to_pt_link1: limit lower=-3.14 upper=3.14 effort=0 velocity=0 -> effort=5.0 velocity=1.5; type revolute -> continuous
- joint pt_link1_to_pt_link2: limit lower=-0.5233333 upper=1.5707963 effort=0 velocity=0 -> lower=-0.5233333 upper=1.5707963 effort=5.0 velocity=1.5
